File: JustWeMini/5Vregulator.kicad_sch (KiCad schematic)
At the start: 15 parts, among them U8 TPS54231

Commit message: Feat: MPN adjusted
Parts:
- C47: value 0.1uF -> 0.1uF 0603
Changed lines of the file:
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@@
       (effects (font (size 1.27 1.27)) hide)
     )
-    (property "Datasheet" "~" (id 3) (at 148.336 52.324 0)
+    (property "Datasheet" "" (id 3) (at 148.336 52.324 0)
       (effects (font (size 1.27 1.27)) hide)
     )
@@
       (effects (font (size 1.27 1.27)) hide)
     )
-    (property "Datasheet" "~" (id 3) (at 48.768 57.15 0)
+    (property "Datasheet" "" (id 3) (at 48.768 57.15 0)
       (effects (font (size 1.27 1.27)) hide)
     )
@@
       (effects (font (size 1.27 1.27)) hide)
     )
-    (property "Datasheet" "~" (id 3) (at 160.02 65.532 0)
+    (property "Datasheet" "" (id 3) (at 160.02 65.532 0)
       (effects (font (size 1.27 1.27)) hide)
     )
@@
       (effects (font (size 1.27 1.27)) hide)
     )
-    (property "Datasheet" "~" (id 3) (at 60.706 61.976 0)
+    (property "Datasheet" "" (id 3) (at 60.706 61.976 0)
       (effects (font (size 1.27 1.27)) hide)
     )
@@
       (effects (font (size 1.27 1.27)) hide)
     )
-    (property "Datasheet" "~" (id 3) (at 83.566 58.928 0)
+    (property "Datasheet" "" (id 3) (at 83.566 58.928 0)
       (effects (font (size 1.27 1.27)) hide)
     )
@@
       (effects (font (size 1.27 1.27)) hide)
     )
-    (property "Datasheet" "~" (id 3) (at 160.02 56.642 0)
+    (property "Datasheet" "" (id 3) (at 160.02 56.642 0)
       (effects (font (size 1.27 1.27)) hide)
     )
@@
       (effects (font (size 1.27 1.27)) hide)
     )
-    (property "Datasheet" "~" (id 3) (at 72.644 61.976 0)
+    (property "Datasheet" "" (id 3) (at 72.644 61.976 0)
       (effects (font (size 1.27 1.27)) hide)
     )
@@
       (effects (font (size 1.27 1.27)) hide)
     )
-    (property "Datasheet" "~" (id 3) (at 169.164 60.96 0)
+    (property "Datasheet" "" (id 3) (at 169.164 60.96 0)
       (effects (font (size 1.27 1.27)) hide)
     )
@@
       (effects (font (size 1.27 1.27)) hide)
     )
-    (property "Datasheet" "~" (id 3) (at 38.608 57.404 0)
+    (property "Datasheet" "" (id 3) (at 38.608 57.404 0)
       (effects (font (size 1.27 1.27)) hide)
     )
@@
       (effects (font (size 1.27 1.27)) (justify left))
     )
-    (property "Value" "0.1uF" (id 1) (at 133.2231 48.0946 0)
+    (property "Value" "0.1uF 0603" (id 1) (at 133.2231 48.0946 0)
       (effects (font (size 1.27 1.27)) (justify left))
     )
@@
       (effects (font (size 1.27 1.27)) hide)
     )
-    (property "Datasheet" "~" (id 3) (at 130.302 46.228 0)
+    (property "Datasheet" "" (id 3) (at 130.302 46.228 0)
       (effects (font (size 1.27 1.27)) hide)
     )
@@
       (effects (font (size 1.27 1.27)) hide)
     )
-    (property "Datasheet" "~" (id 3) (at 60.706 53.086 0)
+    (property "Datasheet" "" (id 3) (at 60.706 53.086 0)
       (effects (font (size 1.27 1.27)) hide)
     )
@@
       (effects (font (size 1.27 1.27)) hide)
     )
-    (property "Datasheet" "~" (id 3) (at 83.566 66.548 0)
+    (property "Datasheet" "" (id 3) (at 83.566 66.548 0)
       (effects (font (size 1.27 1.27)) hide)
     )
@@
       (effects (font (size 1.27 1.27)) hide)
     )
-    (property "Datasheet" "~" (id 3) (at 92.71 61.468 0)
-      (effects (font (size 1.27 1.27)) hide)
-    )
+    (property "Datasheet" "" (id 3) (at 92.71 61.468 0)
+      (effects (font (size 1.27 1.27)) hide)
+    )
