File: JustWeMini/YamarPLC.kicad_sch (KiCad schematic)
At the start: 39 parts, among them U2 DCB1M, Y1 Crystal_GND24_Small

Commit message: Feat: MPN adjusted
Parts:
- C18, C20: value 0.1uF -> 0.1uF 0603
Changed lines of the file:
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@@
     (in_bom yes) (on_board yes) (fields_autoplaced)
     (property "Reference" "C20" (id 0) (at 119.634 45.5253 90))
-    (property "Value" "0.1uF" (id 1) (at 119.634 48.3004 90))
+    (property "Value" "0.1uF 0603" (id 1) (at 119.634 48.3004 90))
     (property "Footprint" "Capacitor_SMD:C_0603_1608Metric" (id 2) (at 119.634 51.054 0)
       (effects (font (size 1.27 1.27)) hide)
@@
       (effects (font (size 1.27 1.27)) (justify right))
     )
-    (property "Value" "0.1uF" (id 1) (at 90.9702 122.2626 0)
+    (property "Value" "0.1uF 0603" (id 1) (at 90.9702 122.2626 0)
       (effects (font (size 1.27 1.27)) (justify right))
     )
